Commit message: Solved error with camera link
Signed-off-by: Juancams <jc.manzanares.serrano@gmail.com>

File: urdf/realsense/_d435.urdf.xacro (robot description, xacro)
@@ -152,4 +152,4 @@
     </xacro:if>
   </xacro:macro>
-  <xacro:gazebo_d435 camera_name="ur5_camera" reference_link="ur5_camera_color_optical_frame" />
+  <xacro:gazebo_d435 camera_name="ur10_camera" reference_link="ur10_camera_gyro_frame" />
 </robot>

File: urdf/ur/ur.urdf.xacro (robot description, xacro)
@@ -139,5 +139,5 @@
   </xacro:ur_robot>
   <xacro:sensor_d435i name="ur10_camera" parent="ur10_wrist_3_link" use_nominal_extrinsics="true">
-    <origin xyz="0 0 0" rpy="0 0 0" />
+    <origin xyz="0 0 0" rpy="0 -1.56 1.56" />
   </xacro:sensor_d435i>
   <xacro:if value="$(arg sim_gazebo)">
