Commit message: gz_ros2_control works
Signed-off-by: Juancams <jc.manzanares.serrano@gmail.com>

File: urdf/ur/ur.ros2_control.xacro (robot description, xacro)
@@ -21,9 +21,10 @@
     non_blocking_read:=true
     keep_alive_count:=2
+    generate_base:=false
     ">
     <ros2_control name="${name}" type="system">
       <hardware>
         <xacro:if value="${sim_gazebo}">
-          <plugin>gz_ros2_control/GazeboSystem</plugin>
+          <plugin>gz_ros2_control/GazeboSimSystem</plugin>
         </xacro:if>
         <xacro:if value="${sim_ignition}">
@@ -160,11 +161,20 @@
         <state_interface name="effort"/>
       </joint>
-      <joint name="${tf_prefix}rail_joint">
-        <command_interface name="position"/>
-        <command_interface name="velocity"/>
-        <state_interface name="position"/>
-        <state_interface name="velocity"/>
-        <state_interface name="effort"/>
-      </joint>
+      <xacro:if value="${generate_base}">
+        <joint name="${tf_prefix}base_joint">
+          <command_interface name="position"/>
+          <command_interface name="velocity"/>
+          <state_interface name="position"/>
+          <state_interface name="velocity"/>
+          <state_interface name="effort"/>
+        </joint>
+        <joint name="${tf_prefix}rail_joint">
+          <command_interface name="position"/>
+          <command_interface name="velocity"/>
+          <state_interface name="position"/>
+          <state_interface name="velocity"/>
+          <state_interface name="effort"/>
+        </joint>
+      </xacro:if>
       <xacro:unless value="${sim_gazebo or sim_ignition}">
         <sensor name="${tf_prefix}tcp_fts_sensor">

File: urdf/ur/ur.urdf.xacro (robot description, xacro)
@@ -146,7 +146,6 @@
     </gazebo>
     <gazebo>
-      <plugin name="gz_ros2_control::GazeboSimROS2ControlPluginl" filename="gz_ros2_control-system">
+      <plugin name="gz_ros2_control::GazeboSimROS2ControlPlugin" filename="gz_ros2_control-system">
         <parameters>$(arg simulation_controllers)</parameters>
-        <controller_manager_prefix_node_name>controller_manager</controller_manager_prefix_node_name>
       </plugin>
       <plugin filename="gz-sim-sensors-system" name="gz::sim::systems::Sensors">

File: urdf/ur/ur_macro.xacro (robot description, xacro)
@@ -60,6 +60,6 @@
     use_fake_hardware:=false
     fake_sensor_commands:=false
-    sim_gazebo:=false
-    sim_ignition:=true
+    sim_gazebo:=true
+    sim_ignition:=false
     headless_mode:=false
     initial_positions:=${dict(shoulder_pan_joint=0.0,shoulder_lift_joint=-1.57,elbow_joint=0.0,wrist_1_joint=-1.57,wrist_2_joint=0.0,wrist_3_joint=0.0)}
@@ -127,4 +127,5 @@
         non_blocking_read="${non_blocking_read}"
         keep_alive_count="${keep_alive_count}"
+        generate_base="${generate_base}"
         />
     </xacro:if>
@@ -279,15 +280,19 @@
     <!-- base_joint fixes base to the environment -->
     <xacro:unless value="${generate_base}">
-      <joint name="${tf_prefix}base_joint" type="fixed">
+      <joint name="${tf_prefix}base_joint" type="prismatic">
         <xacro:insert_block name="origin" />
         <parent link="${parent}" />
         <child link="${tf_prefix}base_link" />
+        <axis xyz="1 0 0"/>
+        <limit lower="0.0" upper="0.0" effort="10" velocity="0.0"/>
       </joint>
     </xacro:unless>
     <xacro:if value="${generate_base}">
-      <joint name="${tf_prefix}base_joint" type="fixed">
+      <joint name="${tf_prefix}base_joint" type="prismatic">
         <xacro:insert_block name="origin" />
         <parent link="${parent}" />
         <child link="${tf_prefix}rail_link" />
+        <axis xyz="1 0 0"/>
+        <limit lower="0.0" upper="0.0" effort="10" velocity="0.0"/>
       </joint>
       <joint name="${tf_prefix}rail_joint" type="prismatic">

Commit message: Solved problem with bases
Signed-off-by: Juancams <jc.manzanares.serrano@gmail.com>

File: urdf/ur/ur.ros2_control.xacro (robot description, xacro)
@@ -162,11 +162,4 @@
       </joint>
       <xacro:if value="${generate_base}">
-        <joint name="${tf_prefix}base_joint">
-          <command_interface name="position"/>
-          <command_interface name="velocity"/>
-          <state_interface name="position"/>
-          <state_interface name="velocity"/>
-          <state_interface name="effort"/>
-        </joint>
         <joint name="${tf_prefix}rail_joint">
           <command_interface name="position"/>

File: urdf/ur/ur_macro.xacro (robot description, xacro)
@@ -280,19 +280,15 @@
     <!-- base_joint fixes base to the environment -->
     <xacro:unless value="${generate_base}">
-      <joint name="${tf_prefix}base_joint" type="prismatic">
+      <joint name="${tf_prefix}base_joint" type="fixed">
         <xacro:insert_block name="origin" />
         <parent link="${parent}" />
         <child link="${tf_prefix}base_link" />
-        <axis xyz="1 0 0"/>
-        <limit lower="0.0" upper="0.0" effort="10" velocity="0.0"/>
       </joint>
     </xacro:unless>
     <xacro:if value="${generate_base}">
-      <joint name="${tf_prefix}base_joint" type="prismatic">
+      <joint name="${tf_prefix}base_joint" type="fixed">
         <xacro:insert_block name="origin" />
         <parent link="${parent}" />
         <child link="${tf_prefix}rail_link" />
-        <axis xyz="1 0 0"/>
-        <limit lower="0.0" upper="0.0" effort="10" velocity="0.0"/>
       </joint>
       <joint name="${tf_prefix}rail_joint" type="prismatic">
